Commit message: update

File: luh_youbot_description/urdf/common.xacro (robot description, xacro)
@@ -1,9 +1,9 @@
 <?xml version="1.0"?>
 <robot>
-	<property name="M_PI" value="3.1415926535897931" />
+	<xacro:property name="M_PI" value="3.1415926535897931" />
 	<!-- Casters -->
-	<property name="cal_caster_fl" value="0.0" />
-	<property name="cal_caster_fr" value="0.0" />
-	<property name="cal_caster_bl" value="0.0" />
-	<property name="cal_caster_br" value="0.0" />
+	<xacro:property name="cal_caster_fl" value="0.0" />
+	<xacro:property name="cal_caster_fr" value="0.0" />
+	<xacro:property name="cal_caster_bl" value="0.0" />
+	<xacro:property name="cal_caster_br" value="0.0" />
 </robot>

File: luh_youbot_description/urdf/sensors/asus_xtion_camera.urdf.xacro (robot description, xacro)
@@ -2,6 +2,6 @@
 <root xmlns:xacro="http://playerstage.sourceforge.net/gazebo/xmlschema/#interface">
   <xacro:include filename="$(find luh_youbot_description)/urdf/sensors/asus_xtion_camera.gazebo.xacro" />
-  <property name="eye_x_offset" value="0.03" />
-  <property name="eye_y_offset" value="0.035" />
+  <xacro:property name="eye_x_offset" value="0.03" />
+  <xacro:property name="eye_y_offset" value="0.035" />
   <xacro:macro name="asus_xtion_eye" params="suffix parent *origin">
 	<link name="${parent}_${suffix}_frame">
@@ -15,5 +15,5 @@
 	  <parent link="${parent}_camera"/>
 	  <child link="${parent}_${suffix}_frame"/>
-	  <insert_block name="origin"/>
+	  <xacro:insert_block name="origin"/>
 	</joint>
   </xacro:macro>
@@ -40,5 +40,5 @@
     </link>
     <joint name="${name}_foot_joint" type="fixed">
-      <insert_block name="origin" />
+      <xacro:insert_block name="origin" />
       <parent link="${parent}"/>
       <child link="${name}_foot_link"/>

File: luh_youbot_description/urdf/sensors/hokuyo_urg04_laser.urdf.xacro (robot description, xacro)
@@ -5,5 +5,5 @@
     <joint name="${name}_hokuyo_urg04_laser_joint" type="fixed">
       <axis xyz="0 1 0" />
-      <insert_block name="origin" />
+      <xacro:insert_block name="origin" />
       <parent link="${parent}_link"/>
       <child link="${name}_link"/>

File: luh_youbot_description/urdf/sensors/kinect_camera.urdf.xacro (robot description, xacro)
@@ -7,5 +7,5 @@
   <xacro:macro name="kinect_camera" params="name parent *origin">
    <joint name="${name}_camera_joint" type="fixed">
-    <insert_block name="origin" />
+    <xacro:insert_block name="origin" />
     <parent link="${parent}" />
     <child link="${name}_camera" />

File: luh_youbot_description/urdf/sensors/microsoft_lifecam.urdf.xacro (robot description, xacro)
@@ -7,5 +7,5 @@
   <xacro:macro name="microsoft_lifecam" params="name parent *origin">
    <joint name="${name}_camera_joint" type="fixed">
-    <insert_block name="origin" />
+    <xacro:insert_block name="origin" />
     <parent link="${parent}" />
     <child link="${name}_camera" />

File: luh_youbot_description/urdf/youbot_arm/arm.urdf.xacro (robot description, xacro)
@@ -6,5 +6,5 @@
         <!-- joint between base_link and arm_0_link -->
         <joint name="${name}_joint_0" type="fixed" >
-            <insert_block name="origin" />
+            <xacro:insert_block name="origin" />
             <parent link="${parent}" />
             <child link="${name}_link_0" />

File: luh_youbot_description/urdf/youbot_arm/limits.urdf.xacro (robot description, xacro)
@@ -2,24 +2,24 @@
 <robot xmlns:xacro="http://ros.org/wiki/xacro">>
 	<!-- common properties -->
-	<property name="M_PI" value="3.1415926535897931" />
-        <property name="threshold" value="0.01" />
+	<xacro:property name="M_PI" value="3.1415926535897931" />
+        <xacro:property name="threshold" value="0.01" />
 	<!-- arm limits positions (deg) -->
-	<property name="joint_1_limit" value="${M_PI * (169 + 169) / 180}" />
-	<property name="joint_2_limit" value="${M_PI * (90 + 65) / 180}" />
-	<property name="joint_3_limit" value="${M_PI * (146 + 151) / 180}" />
-	<property name="joint_4_limit" value="${M_PI * (102.5 + 102.5) / 180}" />
-	<property name="joint_5_limit" value="${M_PI * (167.5 + 167.5) / 180}" />
-        <property name="joint_1_limit_soft" value="${M_PI * (169 + 169) / 180 - threshold}" />
-	<property name="joint_2_limit_soft" value="${M_PI * (90 + 65) / 180 - threshold}" />
-	<property name="joint_3_limit_soft" value="${M_PI * (146 + 151) / 180 - threshold}" />
-	<property name="joint_4_limit_soft" value="${M_PI * (102.5 + 102.5) / 180 - threshold}" />
-	<property name="joint_5_limit_soft" value="${M_PI * (167.5 + 167.5) / 180 - threshold}" />
+	<xacro:property name="joint_1_limit" value="${M_PI * (169 + 169) / 180}" />
+	<xacro:property name="joint_2_limit" value="${M_PI * (90 + 65) / 180}" />
+	<xacro:property name="joint_3_limit" value="${M_PI * (146 + 151) / 180}" />
+	<xacro:property name="joint_4_limit" value="${M_PI * (102.5 + 102.5) / 180}" />
+	<xacro:property name="joint_5_limit" value="${M_PI * (167.5 + 167.5) / 180}" />
+        <xacro:property name="joint_1_limit_soft" value="${M_PI * (169 + 169) / 180 - threshold}" />
+	<xacro:property name="joint_2_limit_soft" value="${M_PI * (90 + 65) / 180 - threshold}" />
+	<xacro:property name="joint_3_limit_soft" value="${M_PI * (146 + 151) / 180 - threshold}" />
+	<xacro:property name="joint_4_limit_soft" value="${M_PI * (102.5 + 102.5) / 180 - threshold}" />
+	<xacro:property name="joint_5_limit_soft" value="${M_PI * (167.5 + 167.5) / 180 - threshold}" />
 	<!-- dynamic properties : mass (kg) Alu data sheet -->
-	<property name="link_0_mass" value="0.845" />
-	<property name="link_1_mass" value="2.412" />
-	<property name="link_2_mass" value="1.155" />
-	<property name="link_3_mass" value="0.934" />
-	<property name="link_4_mass" value="0.877" />
-	<property name="link_5_mass" value="0.251" />
+	<xacro:property name="link_0_mass" value="0.845" />
+	<xacro:property name="link_1_mass" value="2.412" />
+	<xacro:property name="link_2_mass" value="1.155" />
+	<xacro:property name="link_3_mass" value="0.934" />
+	<xacro:property name="link_4_mass" value="0.877" />
+	<xacro:property name="link_5_mass" value="0.251" />
 	<!-- TODO: add inertia tensor-->
 	<xacro:macro name="default_origin">

File: luh_youbot_description/urdf/youbot_base/base.urdf.xacro (robot description, xacro)
@@ -6,19 +6,19 @@
   <xacro:include filename="$(find luh_youbot_description)/urdf/youbot_base/bumper.gazebo.xacro" />
      <!-- simplified box collision geometry for base -->
-      <property name="base_size_x" value="0.570" />
-      <property name="base_size_y" value="0.40" />
-      <property name="base_size_z" value="0.100" />
-      <property name="base_mass" value="22.0" />
-    <property name="wheel_offset_x" value="0.228"  />
-      <property name="wheel_offset_y" value="0.158"  />
-      <property name="wheel_offset_z" value="-0.034" />
-    <property name="wheel_mass" value="0.4" />
-    <property name="wheel_radius" value="0.05" />
-    <property name="wheel_length" value="0.07" />
-    <property name="wheel_joint_damping" value="0.0" />
-    <property name="wheel_joint_friction" value="0.0" />
-    <property name="wheel_joint_effort" value="30" />
-    <property name="wheel_joint_velocity" value="10" />
-    <property name="wheel_joint_safety_k_velocity" value="10.0" />
+      <xacro:property name="base_size_x" value="0.570" />
+      <xacro:property name="base_size_y" value="0.40" />
+      <xacro:property name="base_size_z" value="0.100" />
+      <xacro:property name="base_mass" value="22.0" />
+    <xacro:property name="wheel_offset_x" value="0.228"  />
+      <xacro:property name="wheel_offset_y" value="0.158"  />
+      <xacro:property name="wheel_offset_z" value="-0.034" />
+    <xacro:property name="wheel_mass" value="0.4" />
+    <xacro:property name="wheel_radius" value="0.05" />
+    <xacro:property name="wheel_length" value="0.07" />
+    <xacro:property name="wheel_joint_damping" value="0.0" />
+    <xacro:property name="wheel_joint_friction" value="0.0" />
+    <xacro:property name="wheel_joint_effort" value="30" />
+    <xacro:property name="wheel_joint_velocity" value="10" />
+    <xacro:property name="wheel_joint_safety_k_velocity" value="10.0" />
     <xacro:macro name="youbot_base" params="name namespace">
         <link name="${name}_footprint">

File: luh_youbot_description/urdf/youbot_gripper/gripper.urdf.xacro (robot description, xacro)
@@ -6,5 +6,5 @@
         <!-- joint between arm_7_link and sdh_palm_link -->
         <joint name="${name}_palm_joint" type="fixed" >
-            <insert_block name="origin" />
+            <xacro:insert_block name="origin" />
             <parent link="${parent}" />
             <child link="${name}_palm_link" />

File: luh_youbot_description/urdf/youbot_gripper/limits.urdf.xacro (robot description, xacro)
@@ -2,8 +2,8 @@
 <robot>
     <!-- common properties -->
-    <property name="M_PI" value="3.1415926535897931" />
-        <property name="threshold" value="0.001" />
+    <xacro:property name="M_PI" value="3.1415926535897931" />
+        <xacro:property name="threshold" value="0.001" />
     <!-- fingers limits, values are in meters -->
-    <property name="finger_joint" value="${0.06 / 2.0}" />
-    <property name="finger_joint_soft" value="${(0.06 - threshold) / 2.0}" />
+    <xacro:property name="finger_joint" value="${0.06 / 2.0}" />
+    <xacro:property name="finger_joint_soft" value="${(0.06 - threshold) / 2.0}" />
 </robot>

File: luh_youbot_description/urdf/youbot_plate/plate.urdf.xacro (robot description, xacro)
@@ -4,5 +4,5 @@
 		<!-- joint between arm_7_link and sdh_palm_link -->
 		<joint name="${name}_joint" type="fixed" >
-			<insert_block name="origin" />
+			<xacro:insert_block name="origin" />
 			<parent link="${parent}" />
 			<child link="${name}_link" />
